File: esp_32_sens_RF.kicad_sch (KiCad schematic)
At the start: 21 parts, among them U8 TESEO-LIV3R, U9 BGA725L6E6327FTSA1

Commit message: placement done
placement done, routing left
Parts:
- removed C29: 56p, Capacitor_SMD:C_0402_1005Metric_Pad0.74x0.62mm_HandSolder, symbol Device:C
- AE402: renamed from AE2; footprint (none) -> RF_Antenna:SGGP.25.4.A.02_TAL
- renumbered AE1 to AE401, C26 to C402, C16 to C403, C28 to C404, C27 to C405, C30 to C406, C15 to C407, C32 to C408, C31 to C409, D1 to D401, FL1 to FL401, L3 to L401, L4 to L402, L7 to L403, R18 to R401, R19 to R402, R17 to R403, U8 to U401, U9 to U402
Connections:
- net GND: now also AE401.2 (PCB_Trace); no longer AE401.1 (FEED)
- net feed_pin: now reaches C405.1, D401.2 (A2), L402.2
- net feed_pin: now also AE401.1 (FEED); no longer AE401.2 (PCB_Trace)
- net GPS_VCC: now reaches C407.1, L401.2, U401.6 (VBATT), U401.7 (VCC_IO), U401.8 (VCC)
- net PPS_GPS: no longer names the net of U401.4 (1PPS)
- net RESET_GPS: no longer names the net of U401.9 (SYS_RSTn)
- net WAKEUP_GPS: no longer names the net of U401.5 (Wake-Up)
- no-connect marks 2 -> 5
Other:
- note added: "1575MHz"
- note added: "25x25mm"
- note added: "patch antenna TAOGLAS /SGGP.25.4.A.02 https://cdn.taoglas.com/datasheets/SGGP.25.4.A.02.pdf"
- note removed: "25×25mm"
- note removed: "842MHz"
- note removed: "patch antenna TAOGLAS CGGBP.25.4.A.02 https://www.taoglas.com/datasheets/CGGBP.25.4.A.02.pdf"
- moved on the sheet: AE401
